Commit message: Completed the working solution for robtiq 85 gripper with UR5 rviz launch

File: custom_desciption/urdf/ur5_robotiq/ur5_robotiq.xacro (robot description, xacro)
@@ -1,25 +1,22 @@
 <?xml version="1.0"?>
 <robot xmlns:xacro="http://wiki.ros.org/xacro"
-       name="ur5" >
-  <xacro:arg name="transmission_hw_interface" default="hardware_interface/PositionJointInterface"/>
-  <!-- common stuff -->
-  <xacro:include filename="$(find ur_description)/urdf/common.gazebo.xacro" />
-  <!-- ur5 -->
-  <xacro:include filename="$(find ur_description)/urdf/ur5.urdf.xacro" />
-  <!-- arm -->
-  <xacro:ur5_robot prefix="" joint_limited="false"
-    transmission_hw_interface="$(arg transmission_hw_interface)"
-  />
+       name="ur5_robotiq" >
+<!-- UR5 robot -->
+<xacro:include filename="$(find ur_description)/urdf/ur5_robot.urdf.xacro" />
 <!-- Robotiq gripper -->
-  <xacro:include filename="$(find robotiq_85_description)/urdf/robotiq_85_gripper.urdf.xacro" />
-  <link name="world" />
+<xacro:include filename="$(find robotiq_85_description)/urdf/robotiq_85_gripper.urdf.xacro" />
+ <!-- <link name="world" /> -->
+<!-- Might need this for gazebo
   <joint name="world_joint" type="fixed">
     <parent link="world" />
     <child link = "base_link" />
     <origin xyz="0.0 0.0 0.0" rpy="0.0 0.0 0.0" />
-  </joint>
+  </joint> -->
   <!-- Test the name of the xacro and the position . not sure about either  -->
-  <xacro:robotiq_85_gripper name="robotiq_gripper" parent="ee_link">
-    <origin xyz="0.003 0 0.0052" rpy="0 0 0" />
+   <xacro:robotiq_85_gripper prefix="" parent="ee_link">
+    <origin xyz="0.0 0.0 0.0052" rpy="0 0 0" />
   </xacro:robotiq_85_gripper>
+   <!-- <xacro:robotiq_85_gripper name="robotiq_85_gripper" parent="ee_link">
+    <origin xyz="0.0 0.0 0.0052" rpy="0 0 0" />
+  </xacro:robotiq_85_gripper> -->
 </robot>

File: robotiq_85_description/urdf/robotiq_85_gripper.xacro (robot description, xacro)
@@ -11,29 +11,5 @@
         <origin xyz="0 0 0" rpy="0 0 0"/>
         <parent link="world"/>
-        <child link="gripper_root_link"/>
+        <child link="robotiq_85_base_link"/>
     </joint>
-    <link name="gripper_root_link">
-        <visual>
-            <origin xyz="0 0 0.5" rpy="0 0 0"/>
-            <geometry>
-                <box size="0.1 0.1 1.0"/>
-            </geometry>
-        </visual>
-        <collision>
-            <origin xyz="0 0 0.5" rpy="0 0 0"/>
-            <geometry>
-                <box size="0.1 0.1 1.0"/>
-            </geometry>
-        </collision>
-        <inertial>
-            <mass value="1e2" />
-            <origin xyz="0.0 0.0 0.0" />
-            <inertia ixx = "0.000001" ixy = "0.000000" ixz = "0.000000"
-                     iyx = "0.000000" iyy = "0.000001" iyz = "0.000000"
-                     izx = "0.000000" izy = "0.000000" izz = "0.000001" />
-        </inertial>
-    </link>
-    <xacro:robotiq_85_gripper prefix="" parent="gripper_root_link" >
-        <origin xyz="0.05 0 0.85" rpy="0 0 0"/>
-    </xacro:robotiq_85_gripper>
 </robot>
